Commit message: working on launching DDR robot in gazebo

File: labs/src/lab03/lab03_description/urdf/diff_drive_robot.urdf (robot description, URDF)
Before this commit: robot diff_drive_robot, 5 links, 4 joints
Links:
- removed link back_roller
- removed link front_roller
- added link back_glider; visual sphere radius=0.1
- added link front_glider; visual sphere radius=0.1
Joints:
- removed joint back_roller_joint
- removed joint front_roller_joint
- added joint back_glider_joint: type fixed, parent base_link, child back_glider, origin xyz=0 -0.5 -0.09
- added joint front_glider_joint: type fixed, parent base_link, child front_glider, origin xyz=0 0.5 -0.09
