Commit message: Finished Lab03

File: labs/src/lab03/lab03_description/urdf/ddr.gazebo.xacro (robot description, xacro)
@@ -1,3 +1,96 @@
 <?xml version="1.0"?>
 <robot xmlns:xacro="http://www.ros.org/wiki/xacro" name="diff_drive_robot">
+    <!-- ros_control plugin -->
+    <gazebo>
+      <plugin name="gazebo_ros_control" filename="libgazebo_ros_control.so">
+        <robotNamespace>/ddr</robotNamespace>
+        <robotSimType>gazebo_ros_control/DefaultRobotHWSim</robotSimType>
+      </plugin>
+    </gazebo>
+    <!--
+        Camera Sensor
+    -->
+    <gazebo reference="${camera_name}">
+        <sensor type="camera" name="${camera_name}_sensor">
+            <update_rate>30.0</update_rate>
+            <camera name="${camera_name}_camera">
+                <horizontal_fov>1.3962634</horizontal_fov>
+                <image>
+                    <width>800</width>
+                    <height>800</height>
+                    <format>R8G8B8</format>
+                </image>
+                <clip>
+                    <near>0.02</near>
+                    <far>300</far>
+                </clip>
+                <noise>
+                    <type>gaussian</type>
+                    <mean>0.0</mean>
+                 <stddev>0.007</stddev>
+                </noise>
+            </camera>
+            <!--<plugin name="$camera_controller" filename="libgazebo_ros_openni_kinect.so">
+                <baseline>0.2</baseline>
+                <alwaysOn>true</alwaysOn>
+                <updateRate>1.0</updateRate>
+                <cameraName>${camera_name}_ir</cameraName>
+                <imageTopicName>/${camera_name}/depth/image_raw</imageTopicName>
+                <cameraInfoTopicName>/${camera_name}/depth/camera_info</cameraInfoTopicName>
+                <depthImageTopicName>/${camera_name}/depth/image_raw</depthImageTopicName>
+                <depthImageInfoTopicName>/${camera_name}/depth/camera_info</depthImageInfoTopicName>
+                <pointCloudTopicName>/${camera_name}/depth/points</pointCloudTopicName>
+                <frameName>${camera_name}_frame</frameName>
+                <pointCloudCutoff>0.5</pointCloudCutoff>
+                <distortionK1>0.00000001</distortionK1>
+                <distortionK2>0.00000001</distortionK2>
+                <distortionK3>0.00000001</distortionK3>
+                <distortionT1>0.00000001</distortionT1>
+                <distortionT2>0.00000001</distortionT2>
+                <CxPrime>0</CxPrime>
+                <Cx>0</Cx>
+                <Cy>0</Cy>
+                <focalLength>0</focalLength>
+                <hackBaseline>0</hackBaseline>
+            </plugin>-->
+            <plugin name="camera_controller" filename="libgazebo_ros_camera.so">
+                <alwaysOn>true</alwaysOn>
+                <updateRate>0.0</updateRate>
+                <cameraName>ddr/${camera_name}</cameraName>
+                <imageTopicName>image_raw</imageTopicName>
+                <cameraInfoTopicName>camera_info</cameraInfoTopicName>
+                <frameName>${camera_name}</frameName>
+                <hackBaseline>0.07</hackBaseline>
+                <distortionK1>0.0</distortionK1>
+                <distortionK2>0.0</distortionK2>
+                <distortionK3>0.0</distortionK3>
+                <distortionT1>0.0</distortionT1>
+                <distortionT2>0.0</distortionT2>
+            </plugin>
+        </sensor>
+    </gazebo>
+    <!--
+        Colors
+        http://wiki.ros.org/simulator_gazebo/Tutorials/ListOfMaterials
+    -->
+    <xacro:macro name="gz_black_material" params="name">
+        <gazebo reference="${name}">
+            <material>Gazebo/FlatBlack</material>
+        </gazebo>
+    </xacro:macro>
+    <xacro:macro name="gz_white_material" params="name">
+        <gazebo reference="${name}">
+            <material>Gazebo/White</material>
+        </gazebo>
+    </xacro:macro>
+    <xacro:macro name="gz_blue_material" params="name">
+        <gazebo reference="${name}">
+            <material>Gazebo/Blue</material>
+        </gazebo>
+    </xacro:macro>
+    <xacro:macro name="gz_red_material" params="name">
+        <gazebo reference="${name}">
+            <material>Gazebo/Red</material>
+        </gazebo>
+    </xacro:macro>
 </robot>

File: labs/src/lab03/lab03_description/urdf/ddr.macros.xacro (robot description, xacro)
@@ -1,11 +1,6 @@
 <?xml version="1.0"?>
 <robot xmlns:xacro="http://www.ros.org/wiki/xacro" name="diff_drive_robot">
-    <!--Include Files-->
-    <xacro:include filename="$(find lab03_description)/urdf/ddr.parameters.xacro" />
     <!--
         Macro for creating cylinder inertial
-            mass
-            radius
-            length
     -->
     <xacro:macro name="cylinder_inertial" params="mass radius length">
@@ -13,10 +8,42 @@
             <mass value="${mass}" />
             <inertia
-                ixx="0"
+                ixx="${(1.0 / 12.0) * (3.0 * radius**2 + length**2) * mass}"
+                iyy="${(1.0 / 12.0) * (3.0 * radius**2 + length**2) * mass}"
+                izz="${(1.0 / 12.0) * radius**2 * mass}"
                 ixy="0"
                 ixz="0"
-                iyy="0"
                 iyz="0"
-                izz="0"
+                />
+        </inertial>
+    </xacro:macro>
+    <!--
+        Macro for creating sphere inertial
+    -->
+    <xacro:macro name="sphere_inertial" params="mass radius">
+        <inertial>
+            <mass value="${mass}" />
+            <inertia
+                ixx="${(2.0 / 5.0) * radius**2 * mass}"
+                iyy="${(2.0 / 5.0) * radius**2 * mass}"
+                izz="${(2.0 / 5.0) * radius**2 * mass}"
+                ixy="0"
+                ixz="0"
+                iyz="0"
+                />
+        </inertial>
+    </xacro:macro>
+    <!--
+        Macro for creating cube inertial
+    -->
+    <xacro:macro name="cube_inertial" params="mass x y z">
+        <inertial>
+            <mass value="${mass}" />
+            <inertia
+                ixx="${(1.0 / 12.0) * (y**2 + z**2) * mass}"
+                iyy="${(1.0 / 12.0) * (x**2 + z**2) * mass}"
+                izz="${(1.0 / 12.0) * (y**2 + x**2) * mass}"
+                ixy="0"
+                ixz="0"
+                iyz="0"
                 />
         </inertial>
@@ -30,4 +57,5 @@
     <!--Wheel Macro-->
     <xacro:macro name="wheel" params="name rl_reflection">
+        <xacro:gz_black_material name="${name}" />v
         <link name="${name}">
             <visual>
@@ -49,5 +77,5 @@
         </link>
         <joint name="${name}_joint" type="continuous">
-            <parent link="robot_chassis"/>
+            <parent link="${chassis_name}"/>
             <child link="${name}"/>
             <origin xyz="${rl_reflection * chassis_radius * 0.75} 0 ${wheel_radius * -0.33}"/>
@@ -57,4 +85,5 @@
     <!--Glider Macro-->
     <xacro:macro name="glider" params="name fb_reflection">
+        <xacro:gz_black_material name="${name}" />
         <link name="${name}">
             <visual>
@@ -64,10 +93,45 @@
                 <material name="black"/>
             </visual>
+            <collision>
+                <geometry>
+                    <sphere radius="${glider_radius}" />
+                </geometry>
+            </collision>
+            <xacro:sphere_inertial mass="${glider_mass}"
+                                   radius="${glider_radius}"
+                                   />
         </link>
         <joint name="${name}_joint" type="fixed">
-            <parent link="robot_chassis"/>
+            <parent link="${chassis_name}"/>
             <child link="${name}"/>
             <origin xyz="0 ${fb_reflection * 0.5} -0.09"/>
         </joint>
     </xacro:macro>
+    <!--Camera Macro-->
+    <xacro:macro name="camera" params="name">
+        <xacro:gz_red_material name="${name}" />
+        <link name="${name}">
+            <visual>
+                <geometry>
+                    <box size="${camera_length} ${camera_width} ${camera_height}" />
+                </geometry>
+                <material name="red"/>
+            </visual>
+            <collision>
+                <geometry>
+                    <box size="${camera_length} ${camera_width} ${camera_height}" />
+                </geometry>
+            </collision>
+            <xacro:cube_inertial mass="${camera_mass}"
+                                 x="${camera_length}"
+                                 y="${camera_width}"
+                                 z="${camera_height}"
+                                 />
+        </link>
+        <joint name="${name}_joint" type="fixed">
+            <parent link="${chassis_name}"/>
+            <child link="${name}"/>
+            <origin xyz="0 ${chassis_radius} ${(chassis_height / 2.0) + (camera_height / 2.0)}" />
+        </joint>
+    </xacro:macro>
 </robot>

File: labs/src/lab03/lab03_description/urdf/ddr.main.xacro (robot description, xacro)
@@ -3,19 +3,15 @@
     <!--Include Files-->
     <xacro:include filename="$(find lab03_description)/urdf/ddr.parameters.xacro" />
+    <xacro:include filename="$(find lab03_description)/urdf/ddr.materials.xacro" />
+    <xacro:include filename="$(find lab03_description)/urdf/ddr.gazebo.xacro" />
     <xacro:include filename="$(find lab03_description)/urdf/ddr.macros.xacro" />
-    <xacro:include filename="$(find lab03_description)/urdf/ddr.materials.xacro" />
-    <!--                Arguments
-        <xacro:arg name="chassis_radius" default="0" />
-        <xacro:arg name="chassis_height" default="0" />
-        <xacro:arg name="wheel_radius"   default="0" />
-        <xacro:arg name="glider_radius"  default="0" />
+    <!--
+        Build the robot!
     -->
-    <!--    -->
-    <!--Build the robot!-->
-    <!--    -->
     <!--Base Link-->
     <link name="base_link" />
     <!--Create the chassis and add it to the base link-->
-    <link name="robot_chassis">
+    <xacro:gz_white_material name="${chassis_name}" />
+    <link name="${chassis_name}">
         <visual>
             <xacro:chassis_geometry />
@@ -32,5 +28,5 @@
     <joint name="robot_chassis_joint" type="fixed">
         <parent link="base_link"/>
-        <child link="robot_chassis"/>
+        <child link="${chassis_name}"/>
         <origin xyz="0 0 ${wheel_radius * 1.33 + 0.01}"/>
     </joint>
@@ -38,6 +34,8 @@
     <xacro:wheel name="right_wheel" rl_reflection="1" />
     <xacro:wheel name="left_wheel"  rl_reflection="-1" />
-    Add Gliders
+    <!--Add Gliders-->
     <xacro:glider name="front_glider" fb_reflection="1" />
     <xacro:glider name="back_glider" fb_reflection="-1" />
+    <!--Add Camera-->
+    <xacro:camera name="${camera_name}" />
 </robot>

File: labs/src/lab03/lab03_description/urdf/ddr.parameters.xacro (robot description, xacro)
@@ -14,4 +14,5 @@
     <xacro:property name="vertical_offset" value="${wheel_radius * 1.1}" />
     <!--Chassis properties-->
+    <xacro:property name="chassis_name" value="ddr_chassis" />
     <xacro:property name="chassis_density" value="500.0" />
     <xacro:property name="chassis_radius" value="$(arg chassis_radius)" />
@@ -26,4 +27,11 @@
     <xacro:property name="glider_density" value="200.0" />
     <xacro:property name="glider_radius" value="$(arg glider_radius)" />
-    <xacro:property name="glider_mass" value="${glider_density * (4.0 / 3.0) * pi * glider_radius**3" />
+    <xacro:property name="glider_mass" value="${glider_density * (4.0 / 3.0) * pi * glider_radius**3}" />
+    <!--Camera properties-->
+    <xacro:property name="camera_name" value="rgba_camera" />
+    <xacro:property name="camera_density" value="100.0" />
+    <xacro:property name="camera_length" value="0.2" />
+    <xacro:property name="camera_width" value="0.1" />
+    <xacro:property name="camera_height" value="0.2" />
+    <xacro:property name="camera_mass" value="${camera_density * camera_length * camera_width * camera_height}" />
 </robot>
