Commit message: Adjusting camera position

File: labs/src/lab03/lab03_description/urdf/ddr.macros.xacro (robot description, xacro)
@@ -57,5 +57,5 @@
     <!--Wheel Macro-->
     <xacro:macro name="wheel" params="name rl_reflection">
-        <xacro:gz_black_material name="${name}" />v
+        <xacro:gz_black_material name="${name}" />
         <link name="${name}">
             <visual>
@@ -79,5 +79,5 @@
             <parent link="${chassis_name}"/>
             <child link="${name}"/>
-            <origin xyz="${rl_reflection * chassis_radius * 0.75} 0 ${wheel_radius * -0.33}"/>
+            <origin xyz="${rl_reflection * chassis_radius * 0.75} 0 ${wheel_radius * -0.0}"/>
             <axis xyz="1 0 0"/>
         </joint>
@@ -124,6 +124,6 @@
             </collision>
             <xacro:cube_inertial mass="${camera_mass}"
-                                 x="${camera_length}"
-                                 y="${camera_width}"
+                                 x="${camera_width}"
+                                 y="${camera_length}"
                                  z="${camera_height}"
                                  />
@@ -132,5 +132,5 @@
             <parent link="${chassis_name}"/>
             <child link="${name}"/>
-            <origin xyz="0 ${chassis_radius} ${(chassis_height / 2.0) + (camera_height / 2.0)}" />
+            <origin xyz="0 ${chassis_radius - camera_length} ${(chassis_height / 2.0) + (camera_height / 2.0)}" rpy="0 0 1.571"/>
         </joint>
     </xacro:macro>

File: labs/src/lab03/lab03_description/urdf/ddr.parameters.xacro (robot description, xacro)
@@ -31,6 +31,6 @@
     <xacro:property name="camera_name" value="rgba_camera" />
     <xacro:property name="camera_density" value="100.0" />
-    <xacro:property name="camera_length" value="0.2" />
-    <xacro:property name="camera_width" value="0.1" />
+    <xacro:property name="camera_length" value="0.1" />
+    <xacro:property name="camera_width" value="0.2" />
     <xacro:property name="camera_height" value="0.2" />
     <xacro:property name="camera_mass" value="${camera_density * camera_length * camera_width * camera_height}" />
