Commit message: Moved camera to the front. Added cone world.

File: labs/src/lab04/lab04_description/urdf/ddr.macros.xacro (robot description, xacro)
@@ -132,5 +132,5 @@
             <parent link="${chassis_name}"/>
             <child link="${name}"/>
-            <origin xyz="0 ${chassis_radius - camera_length} ${(chassis_height / 2.0) + (camera_height / 2.0)}" rpy="0 0 1.571"/>
+            <origin xyz="0 ${-(chassis_radius - camera_length)} ${(chassis_height / 2.0) + (camera_height / 2.0)}" rpy="0 0 -1.571"/>
         </joint>
     </xacro:macro>

File: labs/src/lab04/lab04_description/urdf/ddr.main.xacro (robot description, xacro)
@@ -2,8 +2,8 @@
 <robot xmlns:xacro="http://www.ros.org/wiki/xacro" name="diff_drive_robot">
     <!--Include Files-->
-    <xacro:include filename="$(find lab03_description)/urdf/ddr.parameters.xacro" />
-    <xacro:include filename="$(find lab03_description)/urdf/ddr.materials.xacro" />
-    <xacro:include filename="$(find lab03_description)/urdf/ddr.gazebo.xacro" />
-    <xacro:include filename="$(find lab03_description)/urdf/ddr.macros.xacro" />
+    <xacro:include filename="$(find lab04_description)/urdf/ddr.parameters.xacro" />
+    <xacro:include filename="$(find lab04_description)/urdf/ddr.materials.xacro" />
+    <xacro:include filename="$(find lab04_description)/urdf/ddr.gazebo.xacro" />
+    <xacro:include filename="$(find lab04_description)/urdf/ddr.macros.xacro" />
     <!--
         Build the robot!
